File: ScopeFun_PCB/_autosave-file56921512.kicad_sch (KiCad schematic)
At the start: 33 parts, among them IC1 AD9643BCPZ-250, U11 LTC6957-2, U9 SG3225VAN-250Mhz

Commit message: 260410
Connections:
- net CH1+: now also D12.2; no longer D12.1
- net CH1-: now also D12.1; no longer D12.2
- net CH2+: now also D2.4; no longer D2.3
- net CH2-: now also D2.3; no longer D2.4
- net CH1_CM renamed CH_CM
Changed lines of the file:
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@@
 	)
 	(junction
+		(at 48.26 52.07)
+		(diameter 0)
+		(color 0 0 0 0)
+	)
+	(junction
 		(at 210.82 118.11)
 		(diameter 0)
@@
 	)
 	(junction
-		(at 38.1 69.85)
+		(at 40.64 52.07)
 		(diameter 0)
 		(color 0 0 0 0)
 	)
 	(junction
-		(at 40.64 52.07)
+		(at 38.1 69.85)
 		(diameter 0)
 		(color 0 0 0 0)
 	)
 	(junction
-		(at 48.26 49.53)
+		(at 35.56 49.53)
 		(diameter 0)
 		(color 0 0 0 0)
 	)
 	(junction
-		(at 53.34 52.07)
+		(at 40.64 44.45)
 		(diameter 0)
 		(color 0 0 0 0)
@@
 	)
 	(junction
+		(at 53.34 49.53)
+		(diameter 0)
+		(color 0 0 0 0)
+	)
+	(junction
 		(at 173.99 139.7)
 		(diameter 0)
@@
 	)
 	(junction
-		(at 40.64 46.99)
-		(diameter 0)
-		(color 0 0 0 0)
-	)
-	(junction
 		(at 163.83 62.23)
 		(diameter 0)
@@
 	)
 	(junction
+		(at 35.56 46.99)
+		(diameter 0)
+		(color 0 0 0 0)
+	)
+	(junction
 		(at 163.83 59.69)
 		(diameter 0)
@@
 		(color 0 0 0 0)
 	)
-	(junction
-		(at 35.56 44.45)
-		(diameter 0)
-		(color 0 0 0 0)
-	)
-	(junction
-		(at 35.56 49.53)
-		(diameter 0)
-		(color 0 0 0 0)
-	)
 	(no_connect
 		(at 222.25 130.81)
@@
 	(wire
 		(pts
-			(xy 210.82 118.11) (xy 210.82 123.19)
+			(xy 35.56 46.99) (xy 53.34 46.99)
 		)
 		(stroke
@@
 	(wire
 		(pts
-			(xy 157.48 157.48) (xy 157.48 166.37)
+			(xy 210.82 118.11) (xy 210.82 123.19)
 		)
 		(stroke
@@
 	(wire
 		(pts
-			(xy 256.54 147.32) (xy 259.08 147.32)
+			(xy 157.48 157.48) (xy 157.48 166.37)
 		)
 		(stroke
@@
 	(wire
 		(pts
-			(xy 36.83 104.14) (xy 36.83 100.33)
+			(xy 256.54 147.32) (xy 259.08 147.32)
 		)
 		(stroke
@@
 	(wire
 		(pts
-			(xy 233.68 140.97) (xy 233.68 148.59)
+			(xy 36.83 104.14) (xy 36.83 100.33)
 		)
 		(stroke
@@
 	(wire
 		(pts
-			(xy 35.56 29.21) (xy 38.1 29.21)
+			(xy 233.68 140.97) (xy 233.68 148.59)
 		)
 		(stroke
@@
 	(wire
 		(pts
-			(xy 48.26 49.53) (xy 48.26 58.42)
+			(xy 35.56 29.21) (xy 38.1 29.21)
 		)
 		(stroke
@@
 	(wire
 		(pts
-			(xy 35.56 49.53) (xy 48.26 49.53)
-		)
-		(stroke
-			(width 0)
-			(type default)
-		)
-	)
-	(wire
-		(pts
 			(xy 233.68 148.59) (xy 245.11 148.59)
 		)
@@
 	(wire
 		(pts
-			(xy 40.64 52.07) (xy 40.64 58.42)
+			(xy 27.94 142.24) (xy 27.94 143.51)
 		)
 		(stroke
@@
 	(wire
 		(pts
-			(xy 27.94 142.24) (xy 27.94 143.51)
+			(xy 48.26 52.07) (xy 48.26 58.42)
 		)
 		(stroke
@@
 	(wire
 		(pts
-			(xy 40.64 52.07) (xy 53.34 52.07)
+			(xy 35.56 49.53) (xy 53.34 49.53)
 		)
 		(stroke
@@
 	(wire
 		(pts
-			(xy 53.34 52.07) (xy 53.34 58.42)
+			(xy 48.26 52.07) (xy 91.44 52.07)
 		)
 		(stroke
@@
 	(wire
 		(pts
+			(xy 40.64 52.07) (xy 40.64 58.42)
+		)
+		(stroke
+			(width 0)
+			(type default)
+		)
+	)
+	(wire
+		(pts
 			(xy 193.04 124.46) (xy 193.04 125.73)
 		)
@@
 	(wire
 		(pts
-			(xy 31.75 46.99) (xy 40.64 46.99)
+			(xy 40.64 52.07) (xy 48.26 52.07)
 		)
 		(stroke
@@
 	(wire
 		(pts
-			(xy 127 64.77) (xy 134.62 64.77)
+			(xy 40.64 44.45) (xy 48.26 44.45)
 		)
 		(stroke
@@
 	(wire
 		(pts
-			(xy 99.06 142.24) (xy 99.06 143.51)
+			(xy 53.34 49.53) (xy 53.34 58.42)
+		)
+		(stroke
+			(width 0)
+			(type default)
+		)
+	)
+	(wire
+		(pts
+			(xy 127 64.77) (xy 134.62 64.77)
 		)
 		(stroke
@@
 	(wire
 		(pts
-			(xy 40.64 40.64) (xy 40.64 46.99)
+			(xy 99.06 142.24) (xy 99.06 143.51)
 		)
 		(stroke
@@
 	(wire
 		(pts
+			(xy 31.75 52.07) (xy 40.64 52.07)
+		)
+		(stroke
+			(width 0)
+			(type default)
+		)
+	)
+	(wire
+		(pts
 			(xy 210.82 118.11) (xy 207.01 118.11)
 		)
@@
 	(wire
 		(pts
+			(xy 40.64 40.64) (xy 40.64 44.45)
+		)
+		(stroke
+			(width 0)
+			(type default)
+		)
+	)
+	(wire
+		(pts
 			(xy 193.04 124.46) (xy 196.85 124.46)
 		)
@@
 	(wire
 		(pts
-			(xy 48.26 49.53) (xy 91.44 49.53)
-		)
-		(stroke
-			(width 0)
-			(type default)
-		)
-	)
-	(wire
-		(pts
 			(xy 163.83 86.36) (xy 163.83 88.9)
 		)
@@
 	(wire
 		(pts
-			(xy 91.44 66.04) (xy 83.82 66.04)
+			(xy 35.56 40.64) (xy 35.56 46.99)
 		)
 		(stroke
@@
 	(wire
 		(pts
-			(xy 163.83 71.12) (xy 163.83 73.66)
+			(xy 91.44 66.04) (xy 83.82 66.04)
 		)
 		(stroke
@@
 	(wire
 		(pts
-			(xy 35.56 40.64) (xy 35.56 44.45)
+			(xy 163.83 71.12) (xy 163.83 73.66)
 		)
 		(stroke
@@
 	(wire
 		(pts
-			(xy 35.56 49.53) (xy 35.56 58.42)
+			(xy 31.75 49.53) (xy 35.56 49.53)
 		)
 		(stroke
@@
 	(wire
 		(pts
-			(xy 31.75 52.07) (xy 40.64 52.07)
-		)
-		(stroke
-			(width 0)
-			(type default)
-		)
-	)
-	(wire
-		(pts
-			(xy 31.75 44.45) (xy 35.56 44.45)
+			(xy 31.75 44.45) (xy 40.64 44.45)
 		)
 		(stroke
@@
 	(wire
 		(pts
-			(xy 35.56 29.21) (xy 35.56 31.75)
+			(xy 35.56 49.53) (xy 35.56 58.42)
 		)
 		(stroke
@@
 	(wire
 		(pts
-			(xy 64.77 125.73) (xy 64.77 128.27)
+			(xy 35.56 29.21) (xy 35.56 31.75)
 		)
 		(stroke
@@
 	(wire
 		(pts
-			(xy 35.56 44.45) (xy 48.26 44.45)
+			(xy 64.77 125.73) (xy 64.77 128.27)
 		)
 		(stroke
@@
 	(wire
 		(pts
-			(xy 53.34 52.07) (xy 91.44 52.07)
-		)
-		(stroke
-			(width 0)
-			(type default)
-		)
-	)
-	(wire
-		(pts
 			(xy 48.26 29.21) (xy 48.26 31.75)
 		)
@@
 	(wire
 		(pts
-			(xy 31.75 49.53) (xy 35.56 49.53)
-		)
-		(stroke
-			(width 0)
-			(type default)
-		)
-	)
-	(wire
-		(pts
 			(xy 163.83 86.36) (xy 166.37 86.36)
 		)
@@
 	(wire
 		(pts
-			(xy 40.64 46.99) (xy 53.34 46.99)
+			(xy 31.75 46.99) (xy 35.56 46.99)
 		)
 		(stroke
@@
 	(wire
 		(pts
+			(xy 53.34 49.53) (xy 91.44 49.53)
+		)
+		(stroke
+			(width 0)
+			(type default)
+		)
+	)
+	(wire
+		(pts
 			(xy 127 36.83) (xy 134.62 36.83)
 		)
@@
 		)
 	)
-	(global_label "CH1_CM"
+	(global_label "CH_CM"
 		(shape output)
 		(at 82.55 55.88 180)

Commit message: 260412
Connections:
- net CH1+: now also D12.1, D13.4; no longer D12.2, D13.3
- net CH1-: now also D12.2, D13.3; no longer D12.1, D13.4
- net CH_CM renamed CH1_CM
