File: ScopeFun_PCB/file584EFEB1.kicad_sch (KiCad schematic)
At the start: 52 parts, among them J2 SIL6, U12 XC7A35T-FTG256

Commit message: 260417_CHANGED
Parts:
- C190: jlc (none) -> C6119831
Changed lines of the file:
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@@
+			)
+		)
+		(property "jlc" "C6119831"
+			(at 68.58 77.47 0)
+			(hide yes)
+			(show_name no)
+			(do_not_autoplace no)
+			(effects
+				(font
+					(size 1.27 1.27)
+				)
 			)
 		)
