File: ScopeFun_PCB/file58589F31.kicad_sch (KiCad schematic)
At the start: 20 parts

Commit message: 260410
Parts:
- removed C240: C_10u, ScopefunPackagesLibrary:C_0603, symbol ScopefunParts:C_10u
- removed D54: LM431, ScopefunPackagesLibrary:SOT23, symbol ScopefunParts:LM431
- removed R162: R_1.02k, ScopefunPackagesLibrary:R_0603, symbol ScopefunParts:R_1.02k
- removed R165: R_6.8k, ScopefunPackagesLibrary:R_0603, symbol ScopefunParts:R_6.8k
- removed R166: R_22k, ScopefunPackagesLibrary:R_0603, symbol ScopefunParts:R_22k

Commit message: 260417_CHANGED
Other:
- moved on the sheet: C241, C242, C243, D55, D56, D57, R163, R164, R167, R168, R169, R170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
