File: ScopeFun_PCB/file56921512.kicad_sch (KiCad schematic)
At the start: 35 parts, among them IC1 AD9643BCPZ-250, U11 LTC6957-2, U8 KAD5510P-25Q48, U9 SG3225VAN-250Mhz

Commit message: 0326
Parts:
- removed R38: R_10k, ScopefunPackagesLibrary:R_0603, symbol ScopefunParts:R_10k
- removed R66: R_4k7, ScopefunPackagesLibrary:R_0603, symbol ScopefunParts:R_4k7
- removed U8: KAD5510P-25Q48, ScopefunPackagesLibrary:CP-56-2, symbol ScopefunParts:KAD5510P-25Q48
- added C54: C_0.1u, ScopefunPackagesLibrary:C_0603, symbol ScopefunParts:C_0.1u
- added D1, D2: RB851YT2R, ScopefunPackagesLibrary:SOT-543, symbol ScopefunParts:RB851YT2R
- IC1: footprint QFN50P900X900X100-65N-D -> SamacSys_Parts:QFN50P900X900X100-65N-D
Connections:
- net +1.48V: now also C54.1, D2.1, D2.2
- net ADC_RESETN: now also IC1.48 (PDWN)
- net CH1+: now also D12.1, D13.3, IC1.51 (VIN+A)
- net CH1-: now also D12.2, D13.4, IC1.52 (VIN-A)
- net CH1_CM: now also IC1.57 (VCM)
- net CH2+: now also IC1.62 (VIN+B), D1.1, D2.3
- net CH2-: now also IC1.61 (VIN-B), D1.2, D2.4
- net CLK_ADC_N: now also IC1.24 (DCO-)
- net CLK_ADC_P: now also IC1.25 (DCO+)
- net GND: now also C54.2, D1.3, D1.4
- net data1_N: now reaches IC1.11 (D1-)
- net data1_P: now reaches IC1.12 (D1+)
- net data2_N: now reaches IC1.13 (D2-)
- net data2_P: now reaches IC1.14 (D2+)
- net data3_N: now reaches IC1.15 (D3-)
- net data3_P: now reaches IC1.16 (D3+)
- net data4_N: now reaches IC1.17 (D4-)
- net data4_P: now reaches IC1.18 (D4+)
- net data5_N: now reaches IC1.20 (D5-)
- net data5_P: now reaches IC1.21 (D5+)
- net data6_N: now reaches IC1.22 (D6-)
- net data6_P: now reaches IC1.23 (D6+)
- net data7_N: now reaches IC1.26 (D7-)
- net data7_P: now reaches IC1.27 (D7+)
- net data8_N: now reaches IC1.29 (D8-)
- net data8_P: now reaches IC1.30 (D8+)
- net data9_N: now reaches IC1.31 (D9-)
- net data9_P: now reaches IC1.32 (D9+)
- net data10_N: now reaches IC1.33 (D10-)
- net data10_P: now reaches IC1.34 (D10+)
- net data11_N: now reaches IC1.35 (D11-)
- net data11_P: now reaches IC1.36 (D11+)
- net data12_N: now reaches IC1.38 (D12-)
- net data12_P: now reaches IC1.39 (D12+)
- net data13_N: now reaches IC1.40 (D13-_(MSB))
- net data13_P: now reaches IC1.41 (D13+_(MSB))
- net data0_N: now reaches IC1.8 ((LSB)_D0-)
- net data0_P: now reaches IC1.9 ((LSB)_D0+)
- net CH1_ADC_CLK_IN+ renamed ADC_CLK_IN+
- net CH1_ADC_CLK_IN- renamed ADC_CLK_IN-
- no-connect marks 21 -> 11
Other:
- note removed: "180° PHASE BETWEEN ADC1 AND ADC2 CLK_IN"
- moved on the sheet: C58, D12, D13, R39, R68

Commit message: 260410
Parts:
- removed C38: C_22u, ScopefunPackagesLibrary:C_0805, symbol ScopefunParts:C_22u
- removed C53: C_0.1u, ScopefunPackagesLibrary:C_0603, symbol ScopefunParts:C_0.1u
- removed R68: R_2.2k, ScopefunPackagesLibrary:R_0603, symbol ScopefunParts:R_2.2k
- added C38: C_10u, ScopefunPackagesLibrary:C_0603, symbol ScopefunParts:C_0.1u
- C39, C40, C41, C45, C51: value C_0.1u -> C_10u
Connections:
- net +1V8_VA: now also C38.1
- net GND: now also IC1.47 (OEB), C38.2
- no-connect marks 11 -> 13
Other:
- note removed: "HI = NAP LO = NORMAL FT = SLEEP"
- moved on the sheet: C39, C40, C42, C43, C46, C49, C50, L1

Commit message: 260412_1
Connections:
- net CH1+: now also D13.4; no longer D13.3
- net CH1-: now also D13.3; no longer D13.4
- net CH2+: now also D2.4; no longer D2.3
- net CH2-: now also D2.3; no longer D2.4
Changed lines of the file:
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@@
-	)
-	(junction
-		(at 53.34 46.99)
-		(diameter 0)
-		(color 0 0 0 0)
 	)
 	(junction
@@
 	)
 	(junction
-		(at 48.26 49.53)
-		(diameter 0)
-		(color 0 0 0 0)
-	)
-	(junction
-		(at 53.34 52.07)
+		(at 48.26 46.99)
 		(diameter 0)
 		(color 0 0 0 0)
@@
 	)
 	(junction
+		(at 53.34 44.45)
+		(diameter 0)
+		(color 0 0 0 0)
+	)
+	(junction
 		(at 35.56 142.24)
 		(diameter 0)
@@
 	)
 	(junction
+		(at 48.26 52.07)
+		(diameter 0)
+		(color 0 0 0 0)
+	)
+	(junction
 		(at 163.83 78.74)
 		(diameter 0)
@@
 	)
 	(junction
+		(at 53.34 49.53)
+		(diameter 0)
+		(color 0 0 0 0)
+	)
+	(junction
 		(at 66.04 142.24)
 		(diameter 0)
@@
 	(junction
 		(at 163.83 62.23)
-		(diameter 0)
-		(color 0 0 0 0)
-	)
-	(junction
-		(at 48.26 44.45)
 		(diameter 0)
 		(color 0 0 0 0)
@@
 	(wire
 		(pts
-			(xy 48.26 49.53) (xy 48.26 58.42)
-		)
-		(stroke
-			(width 0)
-			(type default)
-		)
-	)
-	(wire
-		(pts
 			(xy 127 54.61) (xy 134.62 54.61)
 		)
@@
 	(wire
 		(pts
-			(xy 35.56 49.53) (xy 48.26 49.53)
+			(xy 35.56 49.53) (xy 53.34 49.53)
 		)
 		(stroke
@@
 	(wire
 		(pts
-			(xy 40.64 52.07) (xy 53.34 52.07)
+			(xy 40.64 52.07) (xy 48.26 52.07)
 		)
 		(stroke
@@
 	(wire
 		(pts
+			(xy 53.34 49.53) (xy 53.34 58.42)
+		)
+		(stroke
+			(width 0)
+			(type default)
+		)
+	)
+	(wire
+		(pts
 			(xy 116.84 142.24) (xy 116.84 143.51)
 		)
@@
 	(wire
 		(pts
-			(xy 53.34 52.07) (xy 53.34 58.42)
-		)
-		(stroke
-			(width 0)
-			(type default)
-		)
-	)
-	(wire
-		(pts
 			(xy 127 72.39) (xy 134.62 72.39)
 		)
@@
 	(wire
 		(pts
-			(xy 48.26 40.64) (xy 48.26 44.45)
-		)
-		(stroke
-			(width 0)
-			(type default)
-		)
-	)
-	(wire
-		(pts
 			(xy 27.94 142.24) (xy 35.56 142.24)
 		)
@@
 	(wire
 		(pts
+			(xy 48.26 52.07) (xy 91.44 52.07)
+		)
+		(stroke
+			(width 0)
+			(type default)
+		)
+	)
+	(wire
+		(pts
 			(xy 35.56 148.59) (xy 35.56 149.86)
 		)
@@
 	(wire
 		(pts
-			(xy 53.34 40.64) (xy 53.34 46.99)
-		)
-		(stroke
-			(width 0)
-			(type default)
-		)
-	)
-	(wire
-		(pts
 			(xy 38.1 69.85) (xy 40.64 69.85)
 		)
@@
 	(wire
 		(pts
-			(xy 48.26 44.45) (xy 91.44 44.45)
+			(xy 35.56 44.45) (xy 53.34 44.45)
 		)
 		(stroke
@@
 	(wire
 		(pts
+			(xy 53.34 49.53) (xy 91.44 49.53)
+		)
+		(stroke
+			(width 0)
+			(type default)
+		)
+	)
+	(wire
+		(pts
 			(xy 210.82 118.11) (xy 207.01 118.11)
 		)
@@
 	(wire
 		(pts
-			(xy 48.26 49.53) (xy 91.44 49.53)
-		)
-		(stroke
-			(width 0)
-			(type default)
-		)
-	)
-	(wire
-		(pts
 			(xy 163.83 86.36) (xy 163.83 88.9)
 		)
@@
 	(wire
 		(pts
-			(xy 53.34 46.99) (xy 91.44 46.99)
-		)
-		(stroke
-			(width 0)
-			(type default)
-		)
-	)
-	(wire
-		(pts
 			(xy 127 80.01) (xy 134.62 80.01)
 		)
@@
 	(wire
 		(pts
+			(xy 48.26 46.99) (xy 91.44 46.99)
+		)
+		(stroke
+			(width 0)
+			(type default)
+		)
+	)
+	(wire
+		(pts
 			(xy 210.82 107.95) (xy 210.82 110.49)
 		)
@@
 	(wire
 		(pts
-			(xy 35.56 44.45) (xy 48.26 44.45)
-		)
-		(stroke
-			(width 0)
-			(type default)
-		)
-	)
-	(wire
-		(pts
 			(xy 127 100.33) (xy 134.62 100.33)
 		)
@@
 	(wire
 		(pts
-			(xy 53.34 52.07) (xy 91.44 52.07)
-		)
-		(stroke
-			(width 0)
-			(type default)
-		)
-	)
-	(wire
-		(pts
 			(xy 48.26 29.21) (xy 48.26 31.75)
 		)
@@
 	(wire
 		(pts
+			(xy 48.26 52.07) (xy 48.26 58.42)
+		)
+		(stroke
+			(width 0)
+			(type default)
+		)
+	)
+	(wire
+		(pts
 			(xy 210.82 149.86) (xy 224.79 149.86)
 		)
@@
 	(wire
 		(pts
+			(xy 53.34 40.64) (xy 53.34 44.45)
+		)
+		(stroke
+			(width 0)
+			(type default)
+		)
+	)
+	(wire
+		(pts
 			(xy 140.97 170.18) (xy 138.43 170.18)
 		)
@@
 	(wire
 		(pts
+			(xy 53.34 44.45) (xy 91.44 44.45)
+		)
+		(stroke
+			(width 0)
+			(type default)
+		)
+	)
+	(wire
+		(pts
 			(xy 31.75 49.53) (xy 35.56 49.53)
 		)
@@
 	(wire
 		(pts
+			(xy 48.26 40.64) (xy 48.26 46.99)
+		)
+		(stroke
+			(width 0)
+			(type default)
+		)
+	)
+	(wire
+		(pts
 			(xy 163.83 86.36) (xy 166.37 86.36)
 		)
@@
 	(wire
 		(pts
-			(xy 40.64 46.99) (xy 53.34 46.99)
-		)
-		(stroke
+			(xy 40.64 46.99) (xy 48.26 46.99)
+		)
+		(stroke

Commit message: 260412_2
Connections:
- net CH1_CM renamed CH_CM

Commit message: 260417_diff_comp
Parts:
- removed C61, C62, C64: C_10n, ScopefunPackagesLibrary:C_0402, symbol ScopefunParts:C_10n_0402
- removed C63: C_0.1u, ScopefunPackagesLibrary:C_0603, symbol ScopefunParts:C_0.1u
- removed R40: R_100, ScopefunPackagesLibrary:R_0402, symbol ScopefunParts:R_100
- removed U11: LTC6957-2, ScopefunPackagesLibrary:12-MSOP, symbol ScopefunParts:LTC6957-2
Connections:
- net OUT2+ is gone; now on net CLK_OUT-: C68.1, R43.2
- net OUT2- is gone; now on net CLK_OUT+: C67.1, R43.1
- net ADC_CLK_IN+: now also IC1.2 (CLK-); no longer IC1.1 (CLK+)
- net ADC_CLK_IN-: now also IC1.1 (CLK+); no longer IC1.2 (CLK-)
- no-connect marks 13 -> 11
Other:
- moved on the sheet: C59, C60, U9

Commit message: 260420
Other:
- moved on the sheet: C38, C39, C40, C41, C42, C43, C44, C45, C46, C49, C50, C51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
