File: ScopeFun_PCB/file56A5A070.kicad_sch (KiCad schematic)
At the start: 83 parts, among them U19 SPX3819, U20 MAX15053, U21 MAX15053, U22 MAX15053, U23 MCP4251, U24 LM2776, U25 MAX15053, U26 MAX15053, U27 SPX3819, U28 TPS72301

Commit message: 260410
Parts:
- removed C106: C_10n, ScopefunPackagesLibrary:C_0603, symbol ScopefunParts:C_10n_100V
- removed C107: C_22u, ScopefunPackagesLibrary:C_0805, symbol ScopefunParts:C_22u
- removed C108: C_10n, ScopefunPackagesLibrary:C_0603, symbol ScopefunParts:C_10n
- removed C115: C_0.1u, ScopefunPackagesLibrary:C_0603, symbol ScopefunParts:C_0.1u
- removed U19: SPX3819, ScopefunPackagesLibrary:SOT23-5_EXAR, symbol ScopefunParts:SPX3819
- removed U23: MCP4251, ScopefunPackagesLibrary:TSSOP14, symbol ScopefunParts:MCP4251
Connections:
- net PWR_EN is gone; now on net +3V3: U24.4 (EN), U27.3 (EN)
- no-connect marks 12 -> 8

Commit message: 260420
Other:
- moved on the sheet: C124, C127, C132, C137, C138, C139, C48, C52, R125, R126, R127, R128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
