File: ScopeFun_PCB/file58597EF4.kicad_sch (KiCad schematic)
At the start: 27 parts, among them U36 IS43TR16256A-125KBL

Commit message: 0326
Parts:
- U36: MFG Part# IS43TR16256A-125KBL -> IS43TR16640B-125JBL
Changed lines of the file:
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@@
 			)
 		)
-		(property "Datasheet" "http://www.issi.com/WW/pdf/43-46TR16256A-85120AL.pdf"
+		(property "Datasheet" "http://www.issi.com/WW/pdf/43-46TR16640B-81280BL.pdf"
 			(at 138.43 134.62 0)
 			(effects
@@
 			)
 		)
-		(property "MFG Part#" "IS43TR16256A-125KBL"
+		(property "MFG Part#" "IS43TR16640B-125JBL"
 			(at 138.43 138.43 0)
 			(effects

Commit message: 260417_CHANGED
Parts:
- U36: value IS43TR16256A-125KBL -> IS43TR16256B-125KBL
Changed lines of the file:
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@@
 			)
 		)
-		(property "Value" "IS43TR16256A-125KBL"
+		(property "Value" "IS43TR16256B-125KBL"
 			(at 138.43 48.26 0)
 			(show_name no)
@@
 			)
 		)
-		(property "Value" "IS43TR16256A-125KBL"
+		(property "Value" "IS43TR16256B-125KBL"
 			(at 254 49.53 0)
 			(show_name no)

Commit message: 260420
Other:
- moved on the sheet: C244, C245, C246, C247, C248, C249, C250, C251, C252, C253, C254, C255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
