File: ScopeFun_PCB/Scopefun_v3.kicad_pcb (KiCad board)
At the start: 6 copper layers, 76.8 x 160.6 mm, 392 parts, among them IC1 AD9643BCPZ-250, J2 SIL6, P1 USB3_TypeB, Q1 BSS138BKS, Q2 BSS138BKS, Q4 DMN6040SSD, U1 ADA4817-1, U12 XC7A35T-FTG256, U13 LTC4360-1, U14 SN74AUP1T17DCKR, U2 ADA4817-1, U20 MAX15053, U21 MAX15053, U22 MAX15053, U24 LM2776, U25 MAX15053, U26 MAX15053, U27 SPX3819, U28 TPS72301, U29 CYUSB3014, U3 AD8337, U30 M24M02-DR, U36 IS43TR16256B-125KBL, U4 AD8337, U5 ADA4932-1, U6 ADA4932-1, U7 LTC6754, U9 SG3225VAN-250Mhz, X1 X_Crystal_19.2Mhz

Commit message: manufactured
Routing:
- net Net-(Q2-G1): track 29.3 -> 29.8 mm
Changed lines of the file:
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@@
 		)
 		(pad_to_mask_clearance 0)
-		(solder_mask_min_width 0.1)
 		(allow_soldermask_bridges_in_footprints no)
 		(tenting
@@
 		(tags "resistor 0805")
 		(property "Reference" "C212"
-			(at -0.1 -3.5 0)
+			(at -1.5 -1 0)
 			(layer "B.SilkS")
 			(effects
@@
 		(tags "resistor 0603")
 		(property "Reference" "C215"
-			(at -0.1 -3.5 0)
+			(at 0.2 -2.1 90)
 			(layer "B.SilkS")
 			(effects
@@
 		(tags "resistor 0603")
 		(property "Reference" "C221"
-			(at 1.43 -0.6 180)
+			(at 0.2 3.2 180)
 			(layer "B.SilkS")
 			(effects
@@
 		(tags "resistor 0805")
 		(property "Reference" "C100"
-			(at 0.22 -2.62 0)
+			(at 0.76 -2.57 0)
 			(layer "B.SilkS")
 			(effects
@@
 		(tags "resistor 0603")
 		(property "Reference" "R107"
-			(at -1.54 0 0)
+			(at -2.34 0.2 0)
 			(layer "B.SilkS")
 			(effects
@@
 		(at 78.94 140.25 90)
 		(property "Reference" "C119"
-			(at 1.4 4 0)
+			(at 2.15 0.16 0)
 			(layer "B.SilkS")
 			(effects
@@
 		(tags "resistor 0603")
 		(property "Reference" "C112"
-			(at -1.47 1.23 0)
+			(at -2.27 -1.67 0)
 			(layer "B.SilkS")
 			(effects
@@
 		(tags "resistor 0603")
 		(property "Reference" "R110"
-			(at -1.1 2.3 0)
+			(at -1.75 3.44 90)
 			(layer "B.SilkS")
 			(effects
@@
 		(tags "resistor 0603")
 		(property "Reference" "R104"
-			(at 1.73 0.32 0)
+			(at 1.25 1.84 90)
 			(layer "B.SilkS")
 			(effects
@@
 		(tags "resistor 0603")
 		(property "Reference" "R111"
-			(at 0.19 1.55 0)
+			(at 1.75 -3.44 90)
 			(layer "B.SilkS")
 			(effects
@@
 		(tags "resistor 0603")
 		(property "Reference" "C116"
-			(at -0.2 3.6 0)
+			(at -1.55 3.44 90)
 			(layer "B.SilkS")
 			(effects
@@
 		(tags "MURATA Inductor")
 		(property "Reference" "L2"
-			(at -0.025 3.625 0)
+			(at -3.13 1.51 0)
 			(layer "B.SilkS")
 			(effects
@@
 	)
 	(segment
+		(start 47.397721 66.64149)
+		(end 47.387221 66.65199)
+		(width 0.15)
+		(layer "B.Cu")
+		(net "Net-(Q2-G1)")
+	)
+	(segment
+		(start 59.85 72.45)
+		(end 54.04149 66.64149)
+		(width 0.15)
+		(layer "B.Cu")
+		(net "Net-(Q2-G1)")
+	)
+	(segment
 		(start 44.49149 66.64149)
 		(end 44.375 66.525)
@@
 	)
 	(segment
-		(start 53.161311 66.64149)
+		(start 59.85 82.55)
+		(end 59.85 72.45)
+		(width 0.15)
+		(layer "B.Cu")
+		(net "Net-(Q2-G1)")
+	)
+	(segment
+		(start 47.002279 66.64149)
 		(end 44.49149 66.64149)
-		(width 0.127)
+		(width 0.15)
 		(layer "B.Cu")
 		(net "Net-(Q2-G1)")
 	)
 	(segment
-		(start 59.85 82.55)
-		(end 59.85 73.330179)
-		(width 0.127)
+		(start 47.012779 66.65199)
+		(end 47.002279 66.64149)
+		(width 0.15)
 		(layer "B.Cu")
 		(net "Net-(Q2-G1)")
 	)
 	(segment
-		(start 59.85 73.330179)
-		(end 53.161311 66.64149)
-		(width 0.127)
+		(start 47.387221 66.65199)
+		(end 47.012779 66.65199)
+		(width 0.15)
+		(layer "B.Cu")
+		(net "Net-(Q2-G1)")
+	)
+	(segment
+		(start 54.04149 66.64149)
+		(end 47.397721 66.64149)
+		(width 0.15)
 		(layer "B.Cu")
 		(net "Net-(Q2-G1)")
