File: ScopeFun_PCB/Scopefun_v3.kicad_pcb (KiCad board)
At the start: 6 copper layers, 76.8 x 160.6 mm, 392 parts, among them IC1 AD9643BCPZ-250, J2 SIL6, P1 USB3_TypeB, Q1 BSS138BKS, Q2 BSS138BKS, Q4 DMN6040SSD, U1 ADA4817-1, U12 XC7A35T-FTG256, U13 LTC4360-1, U14 SN74AUP1T17DCKR, U2 ADA4817-1, U20 MAX15053, U21 MAX15053, U22 MAX15053, U24 LM2776, U25 MAX15053, U26 MAX15053, U27 SPX3819, U28 TPS72301, U29 CYUSB3014, U3 AD8337, U30 M24M02-DR, U36 IS43TR16256B-125KBL, U4 AD8337, U5 ADA4932-1, U6 ADA4932-1, U7 LTC6754, U9 SG3225VAN-250Mhz, X1 X_Crystal_19.2Mhz

Commit message: 0527_dacchange
Parts:
- removed C35, C36, C37: C_0.1u, ScopefunPackagesLibrary:C_0603
- removed D11: 1N4148W, ScopefunPackagesLibrary:SOD123
- removed R31: R_499R, ScopefunPackagesLibrary:R_0603
- removed R36, R37: R_6.8k, ScopefunPackagesLibrary:R_0603
- removed R56: R_100, ScopefunPackagesLibrary:R_0402
- removed RE7: G6K-2F-Y-DC4.5, ScopefunPackagesLibrary:G6K-2F-Y
- added C232: C_2.2u, ScopefunPackagesLibrary:C_0603, F.Cu at (69.0, 99.5)
- added C233: C_2.2u, ScopefunPackagesLibrary:C_0603, F.Cu at (62.0, 100.0)
- added C234: C_0.1u, ScopefunPackagesLibrary:C_0603, F.Cu at (54.4, 93.0)
- added C235: C_0.1u, ScopefunPackagesLibrary:C_0603, F.Cu at (54.6, 87.5)
- added C236: C_0.1u, ScopefunPackagesLibrary:C_0603, F.Cu at (59.8, 103.8)
- added C237: C_10n, ScopefunPackagesLibrary:C_0402, F.Cu at (58.0, 105.4)
- added C238: C_0.1u, ScopefunPackagesLibrary:C_0603, F.Cu at (37.7, 96.0)
- added C239: C_0.1u, ScopefunPackagesLibrary:C_0603, F.Cu at (24.7, 92.8)
- added D53: MCP1501-18, ScopefunPackagesLibrary:SOT23-6, F.Cu at (65.8, 99.6)
- added R152: R_1.02k, ScopefunPackagesLibrary:R_0603, F.Cu at (65.8, 96.4)
- added R153: R_56R, ScopefunPackagesLibrary:R_0603, F.Cu at (60.0, 99.9)
- added R154: R_1.02k, ScopefunPackagesLibrary:R_0603, F.Cu at (58.0, 93.0)
- added R155: R_1.02k, ScopefunPackagesLibrary:R_0603, F.Cu at (58.0, 87.5)
- added R156: R_1.02k, ScopefunPackagesLibrary:R_0603, F.Cu at (61.1, 95.4)
- added R157: R_1.02k, ScopefunPackagesLibrary:R_0603, F.Cu at (62.4, 85.8)
- added R158: R_1.02k, ScopefunPackagesLibrary:R_0603, F.Cu at (56.2, 93.0)
- added R159: R_1.02k, ScopefunPackagesLibrary:R_0603, F.Cu at (56.3, 87.5)
- added R160: R_1.02k, ScopefunPackagesLibrary:R_0603, F.Cu at (56.8, 108.9)
- added R161: R_1.02k, ScopefunPackagesLibrary:R_0603, F.Cu at (56.8, 110.6)
- added U33: MAX5501, ScopefunPackagesLibrary:SSOP20, F.Cu at (63.4, 109.3)
- added U34: OPA692, ScopefunPackagesLibrary:SOT23-6, F.Cu at (40.4, 96.0)
- added U35: OPA692, ScopefunPackagesLibrary:SOT23-6, F.Cu at (25.7, 96.7)
- U7: value LTC6754 -> AZ4558C; footprint ScopefunPackagesLibrary:SC70-6 -> ScopefunPackagesLibrary:SOIC8
- moved U7 22.3 mm to (62.5, 90.8), turned to 90 degrees
- moved R59 18.7 mm to (85.2, 94.2)
- moved R1 18.6 mm to (77.4, 94.2)
- moved R6 18.6 mm to (74.2, 94.2)
- moved R7 18.6 mm to (75.8, 94.2)
- moved R8 18.6 mm to (72.6, 94.2)
- moved R3 18.6 mm to (80.1, 94.2)
- moved R60 18.6 mm to (83.5, 94.2)
- moved R2 18.5 mm to (81.8, 94.2)
- moved C241 8.20 mm to (77.5, 72.0)
- moved R163 8.20 mm to (77.5, 73.6)
- moved R168 8.20 mm to (74.2, 77.8)
- moved R170 8.20 mm to (67.0, 77.8)
- moved D55 8.20 mm to (77.5, 77.9)
- moved R167 8.20 mm to (77.5, 75.2)
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Connections:
- U12 pad M4: unconnected-(U12B-IO_L1N_T0_34-PadM4) -> DASCLK
- U12 pad N3: unconnected-(U12B-IO_L3P_T0_DQS_34-PadN3) -> DASDIN
- U12 pad N4: unconnected-(U12B-IO_L6N_T0_VREF_34-PadN4) -> DASYNC
- U12 pad R6: AN_TRIG_P -> unconnected-(U12A-IO_L24P_T3_A01_D17_14-PadR6)
- U12 pad R7: AN_TRIG_N -> unconnected-(U12A-IO_L24N_T3_A00_D16_14-PadR7)
- U12 pad T12: AN_TRIG_LEVEL -> unconnected-(U12A-IO_L15N_T2_DQS_DOUT_CSO_B_14-PadT12)
- U4 pad 3: Net-(U4-INPP) -> /ANALOG INPUTS/CH2_VGA
- U7 pad 1: AN_TRIG_P -> Net-(U7A-~)
- U7 pad 2: GND -> Net-(U7A--)
- U7 pad 3: Net-(U7-+) -> CH2_GAIN_ADJ
- U7 pad 4: /GAIN, OFFSET/AN_TRIG -> -Va
- U7 pad 5: +3V3 -> CH1_GAIN_ADJ
- U7 pad 6: AN_TRIG_N -> Net-(U7B--)
Routing:
- net RE7: track 78.8 -> 0.00 mm, vias 3 -> 0
- net LED[3]: track 65.7 -> 0.00 mm, vias 3 -> 0
- net CH2_GND: track 63.1 -> 0.00 mm, vias 2 -> 0
- net Net-(LED3-A): track 61.5 -> 2.77 mm, vias 1 -> 0
- net LED[2]: track 57.8 -> 0.00 mm, vias 2 -> 0
- net CH2_DC: track 57.0 -> 0.00 mm, vias 2 -> 0
- net CH1_GND: track 56.8 -> 0.00 mm, vias 2 -> 0
- net CH2_K: track 56.6 -> 0.00 mm, vias 2 -> 0
- net Net-(R3-Pad2): track 55.1 -> 0.00 mm, vias 2 -> 0
- net CH1_DC: track 54.9 -> 0.00 mm, vias 2 -> 0
- net CH1_K: track 53.4 -> 0.00 mm, vias 2 -> 0
- net Net-(LED2-A): track 51.5 -> 2.84 mm, vias 2 -> 0
- net Net-(R2-Pad2): track 42.6 -> 0.00 mm, vias 2 -> 0
- net AN_TRIG_LEVEL: track 40.1 -> 0.00 mm, vias 2 -> 0
- net AN_TRIG_P: track 31.1 -> 0.00 mm
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
Commit message: 0531
Parts:
- moved R1 30.7 mm to (58.8, 118.5)
- moved R6 30.7 mm to (55.6, 118.5)
- moved R7 30.7 mm to (57.2, 118.5)
- moved R8 30.7 mm to (54.0, 118.5)
- moved U35 16.4 mm to (42.1, 97.5)
- moved C239 14.8 mm to (39.3, 95.0)
- moved U34 14.0 mm to (26.4, 96.8)
- moved C238 12.7 mm to (25.4, 92.8)
- moved R59 7.61 mm to (77.6, 93.9)
- moved R2 7.61 mm to (74.2, 94.0)
- moved R3 7.61 mm to (72.5, 94.0)
- moved R60 7.61 mm to (75.9, 94.0)
- moved C236 0.70 mm to (59.0, 103.8)
- moved C237 0.10 mm to (58.0, 105.4)
Routing:
- net Net-(LED3-A): track 2.77 -> 81.4 mm, vias 0 -> 1
- net Net-(R3-Pad2): track 0.00 -> 76.9 mm, vias 0 -> 2
- net Net-(Q1-G2): track 0.00 -> 63.0 mm, vias 0 -> 2
- net Net-(LED2-A): track 2.84 -> 64.3 mm, vias 0 -> 1
- net Net-(Q2-G2): track 0.00 -> 58.5 mm, vias 0 -> 2
- net Net-(Q2-G1): track 0.00 -> 58.0 mm, vias 0 -> 2
- net Net-(R2-Pad2): track 0.00 -> 55.8 mm, vias 0 -> 2
- net Net-(Q1-G1): track 0.00 -> 55.2 mm, vias 0 -> 2
- net LED[2]: track 0.00 -> 53.5 mm, vias 0 -> 3
- net LED[3]: track 0.00 -> 53.4 mm, vias 0 -> 2
- net CH1_DC: track 0.00 -> 51.0 mm, vias 0 -> 3
- net CH2_DC: track 0.00 -> 50.4 mm, vias 0 -> 2
- net DASCLK: track 0.00 -> 37.7 mm, vias 0 -> 3
- net DASDIN: track 0.00 -> 34.4 mm, vias 0 -> 2
- net DASYNC: track 0.00 -> 29.9 mm, vias 0 -> 2
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