File: ScopeFun_PCB/Scopefun_v3.kicad_pcb (KiCad board)
At the start: 6 copper layers, 76.8 x 160.6 mm, 405 parts, among them IC1 AD9643BCPZ-250, J2 SIL6, P1 USB3_TypeB, Q1 BSS138BKS, Q2 BSS138BKS, Q4 DMN6040SSD, U1 ADA4817-1, U12 XC7A35T-FTG256, U13 LTC4360-1, U14 SN74AUP1T17DCKR, U2 ADA4817-1, U20 MAX15053, U21 MAX15053, U22 MAX15053, U24 LM2776, U25 MAX15053, U26 MAX15053, U27 SPX3819, U28 TPS72301, U29 CYUSB3014, U3 AD8337, U30 M24M02-DR, U33 MAX5501, U34 OPA692, U35 OPA692, U36 IS43TR16256B-125KBL, U4 AD8337, U5 ADA4932-1, U6 ADA4932-1, U7 AZ4558C, U9 SG3225VAN-250Mhz, X1 X_Crystal_19.2Mhz

Commit message: 260601
Parts:
- moved C38 0.71 mm to (34.2, 120.4)
- moved C44 0.71 mm to (34.2, 118.9)
Changed lines of the file:
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@@
 	(footprint "ScopefunPackagesLibrary:C_0603"
 		(layer "F.Cu")
-		(at 34.27 121.11 -90)
+		(at 34.25 120.4 -90)
 		(descr "Resistor SMD 0603, reflow soldering, Vishay (see dcrcw.pdf)")
 		(tags "resistor 0603")
 		(property "Reference" "C38"
-			(at 1.22 2.69 90)
+			(at -0.1 4.25 90)
 			(layer "F.SilkS")
 			(effects
@@
 	(footprint "ScopefunPackagesLibrary:C_0603"
 		(layer "F.Cu")
-		(at 34.27 119.61 -90)
+		(at 34.25 118.9 -90)
 		(descr "Resistor SMD 0603, reflow soldering, Vishay (see dcrcw.pdf)")
 		(tags "resistor 0603")
 		(property "Reference" "C44"
-			(at -0.1 2.67 90)
+			(at 0.2 2.85 90)
 			(layer "F.SilkS")
 			(effects
@@
 	)
 	(segment
-		(start 33.52 121.11)
-		(end 32.81 121.11)
+		(start 33.5 120.4)
+		(end 32.79 120.4)
 		(width 0.2)
 		(layer "F.Cu")
@@
 	)
 	(segment
-		(start 33.52 119.61)
-		(end 32.74 119.61)
+		(start 33.5 118.9)
+		(end 32.72 118.9)
 		(width 0.2)
 		(layer "F.Cu")
@@
 	)
 	(segment
-		(start 32.81 121.11)
-		(end 32.79 121.13)
-		(width 0.2)
-		(layer "F.Cu")
-		(net "GND")
-	)
-	(segment
 		(start 37.6 155.1)
 		(end 38 155.5)
@@
 	)
 	(segment
-		(start 32.74 119.61)
-		(end 32.73 119.62)
-		(width 0.2)
-		(layer "F.Cu")
-		(net "GND")
-	)
-	(segment
 		(start 24.325 133.2)
 		(end 24.325 132.5)
@@
 	)
 	(via
-		(at 32.79 121.13)
+		(at 32.77 120.42)
 		(size 0.4)
 		(drill 0.2)
@@
 	)
 	(via
-		(at 32.73 119.62)
+		(at 32.71 118.91)
 		(size 0.4)
 		(drill 0.2)
@@
 	)
 	(segment
-		(start 37.925 118.65)
-		(end 39.26 119.985)
+		(start 33.55 117.9)
+		(end 37.1 117.9)
 		(width 0.2)
 		(layer "F.Cu")
@@
 	)
 	(segment
-		(start 39.26 119.985)
-		(end 39.26 120.56)
+		(start 37.1 117.9)
+		(end 39.26 120.06)
 		(width 0.2)
 		(layer "F.Cu")
@@
 	)
 	(segment
-		(start 31.74 114.11)
-		(end 31.74 116.09)
+		(start 32.75 117.1)
+		(end 33.55 117.9)
 		(width 0.2)
 		(layer "F.Cu")
@@
 	)
 	(segment
-		(start 34.3 118.65)
-		(end 37.925 118.65)
+		(start 31.74 114.11)
+		(end 31.74 116.09)
 		(width 0.2)
 		(layer "F.Cu")
@@
 	)
 	(segment
+		(start 39.26 120.06)
+		(end 39.26 120.56)
+		(width 0.2)
+		(layer "F.Cu")
+		(net "/ADC/CH2+")
+	)
+	(segment
 		(start 31.77 110.17)
 		(end 30.99 110.95)
@@
 	)
 	(segment
-		(start 32.75 117.1)
-		(end 34.3 118.65)
-		(width 0.2)
-		(layer "F.Cu")
-		(net "/ADC/CH2+")
-	)
-	(segment
 		(start 46.46 120.71)
 		(end 46.46 121.26)
@@
 		)
 		(min_thickness 0.25)
-		(fill yes
+		(fill
 			(thermal_gap 0.5)
 			(thermal_bridge_width 0.5)
@@
 		(polygon
 			(pts
-				(xy 34.69 119.17) (xy 34.7 121.54) (xy 35.5 121.55) (xy 36.3 120.85) (xy 38.88 120.85) (xy 38.89 119.86)
-				(xy 38.66 119.67) (xy 35.83 119.58) (xy 35.4 119.21)
+				(xy 34.69 119.17) (xy 34.691795 121.103652) (xy 35.997908 121.119979) (xy 36.3 120.85) (xy 38.88 120.85)
+				(xy 38.89 119.86) (xy 38.66 119.67) (xy 35.83 119.58) (xy 35.4 119.21)
 			)
 		)

Commit message: 260610_runable
Parts:
- turned C238 to 180 degrees
Routing:
- net Net-(U34-IN+): track 3.91 -> 48.3 mm, vias 0 -> 2
- net Net-(U35-IN+): track 2.08 -> 33.2 mm, vias 0 -> 2
- net GND: track 308.2 -> 308.9 mm, vias 368 -> 367
Changed lines of the file:
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@@
 	(footprint "ScopefunPackagesLibrary:C_0603"
 		(layer "F.Cu")
-		(at 25.4 92.85)
+		(at 25.4 92.85 180)
 		(descr "Resistor SMD 0603, reflow soldering, Vishay (see dcrcw.pdf)")
 		(tags "resistor 0603")
@@
 		)
 		(property "MFG Part#" "C0603C104K4RACTU"
-			(at 0 0 0)
+			(at 0 0 180)
 			(unlocked yes)
 			(layer "F.Fab")
@@
 		(duplicate_pad_numbers_are_jumpers no)
 		(fp_line
-			(start -0.7 -1.35)
-			(end 0.7 -1.35)
+			(start 0.7 1.35)
+			(end -0.7 1.35)
 			(stroke
 				(width 0.2032)
@@
 		)
 		(fp_line
-			(start -0.7 1.35)
-			(end -0.7 -1.35)
+			(start 0.7 -1.35)
+			(end 0.7 1.35)
 			(stroke
 				(width 0.2032)
@@
 		)
 		(fp_line
-			(start 0.7 -1.35)
-			(end 0.7 1.35)
+			(start -0.7 1.35)
+			(end -0.7 -1.35)
 			(stroke
 				(width 0.2032)
@@
 		)
 		(fp_line
-			(start 0.7 1.35)
-			(end -0.7 1.35)
+			(start -0.7 -1.35)
+			(end 0.7 -1.35)
 			(stroke
 				(width 0.2032)
@@
 		)
 		(pad "1" smd rect
-			(at 0 -0.75 270)
+			(at 0 -0.75 90)
 			(size 0.635 0.889)
 			(layers "F.Cu" "F.Mask" "F.Paste")
@@
 		)
 		(pad "2" smd rect
-			(at 0 0.75 270)
+			(at 0 0.75 90)
 			(size 0.635 0.889)
 			(layers "F.Cu" "F.Mask" "F.Paste")
@@
 	)
 	(segment
+		(start 25.4 91.05)
+		(end 25.05 90.7)
+		(width 0.5)
+		(layer "F.Cu")
+		(net "GND")
+	)
+	(segment
 		(start 38.4 155.1)
 		(end 38.8 155.5)
@@
 	)
 	(segment
-		(start 25.4 93.6)
-		(end 25.4 94.4)
-		(width 0.5)
-		(layer "F.Cu")
-		(net "GND")
-	)
-	(segment
 		(start 54.2 161.526)
 		(end 54.2 160.95)
@@
 	)
 	(segment
+		(start 25.4 92.1)
+		(end 25.4 91.05)
+		(width 0.5)
+		(layer "F.Cu")
+		(net "GND")
+	)
+	(segment
 		(start 77.90775 186.16275)
 		(end 77.90775 184.7076)
@@
 	)
 	(via
-		(at 25.4 94.4)
-		(size 0.5)
-		(drill 0.25)
-		(layers "F.Cu" "B.Cu")
-		(net "GND")
-	)
-	(via
 		(at 71.15 153.5)
 		(size 0.5)
@@
 	)
 	(segment
-		(start 24.72851 92.77149)
-		(end 24.72851 94.77851)
+		(start 53.5 96.2)
+		(end 56.125 98.825)
 		(width 0.2)
 		(layer "F.Cu")
@@
 	)
 	(segment
-		(start 24.72851 94.77851)
+		(start 24.7 93.6)
+		(end 25.4 93.6)
+		(width 0.2)
+		(layer "F.Cu")
+		(net "Net-(U34-IN+)")
+	)
+	(segment
+		(start 24.85 95.45)
 		(end 25.4 95.45)
 		(width 0.2)
@@
 	)
 	(segment
-		(start 25.4 92.1)
-		(end 24.72851 92.77149)
+		(start 56.125 98.825)
+		(end 56.125 108.775)
+		(width 0.2)
+		(layer "F.Cu")
+		(net "Net-(U34-IN+)")
+	)
+	(segment
+		(start 24.5 95.1)
+		(end 24.85 95.45)
+		(width 0.2)
+		(layer "F.Cu")
+		(net "Net-(U34-IN+)")
+	)
+	(segment
+		(start 24.5 93.8)
+		(end 24.7 93.6)
+		(width 0.2)
+		(layer "F.Cu")
+		(net "Net-(U34-IN+)")
+	)
+	(segment
+		(start 24.5 94.3)
+		(end 24.5 95.1)
+		(width 0.2)
+		(layer "F.Cu")
+		(net "Net-(U34-IN+)")
+	)
+	(segment
+		(start 56.125 108.775)
+		(end 56 108.9)
 		(width 0.2)
 		(layer "F.Cu")
@@
 	)
 	(segment
+		(start 24.5 94.3)
+		(end 24.5 93.8)
+		(width 0.2)
+		(layer "F.Cu")
+		(net "Net-(U34-IN+)")
+	)
+	(via
+		(at 53.5 96.2)
+		(size 0.5)
+		(drill 0.25)
+		(layers "F.Cu" "B.Cu")
+		(net "Net-(U34-IN+)")
+	)
+	(via
+		(at 24.5 94.3)
+		(size 0.5)
+		(drill 0.25)
+		(layers "F.Cu" "B.Cu")
+		(net "Net-(U34-IN+)")
+	)
+	(segment
+		(start 29.4 92.9)
+		(end 38.825434 92.9)
+		(width 0.2)
+		(layer "B.Cu")
+		(net "Net-(U34-IN+)")
+	)
+	(segment
+		(start 39.774566 92.9)
+		(end 50.2 92.9)
+		(width 0.2)
+		(layer "B.Cu")
+		(net "Net-(U34-IN+)")
+	)
+	(segment
+		(start 39.102424 93.17699)
+		(end 39.497576 93.17699)
+		(width 0.2)
+		(layer "B.Cu")
+		(net "Net-(U34-IN+)")
+	)
+	(segment
+		(start 28 94.3)
+		(end 24.5 94.3)
+		(width 0.2)
+		(layer "B.Cu")
+		(net "Net-(U34-IN+)")
+	)
+	(segment
+		(start 39.497576 93.17699)
+		(end 39.774566 92.9)
+		(width 0.2)
+		(layer "B.Cu")
+		(net "Net-(U34-IN+)")
+	)
+	(segment
+		(start 38.825434 92.9)
+		(end 39.102424 93.17699)
+		(width 0.2)
+		(layer "B.Cu")
+		(net "Net-(U34-IN+)")
+	)
+	(segment
+		(start 29.4 92.9)
+		(end 28 94.3)
+		(width 0.2)
+		(layer "B.Cu")
+		(net "Net-(U34-IN+)")
+	)
+	(segment
+		(start 50.2 92.9)
+		(end 53.5 96.2)
+		(width 0.2)
+		(layer "B.Cu")
+		(net "Net-(U34-IN+)")
+	)
+	(segment
+		(start 41.15 96.55)
+		(end 41.15 96.15)
+		(width 0.2)
+		(layer "F.Cu")
+		(net "Net-(U35-IN+)")
+	)
+	(segment
+		(start 56 110.6)
+		(end 55.11119 109.71119)
+		(width 0.2)
+		(layer "F.Cu")
+		(net "Net-(U35-IN+)")
+	)
+	(segment
 		(start 41.1 96.2)
 		(end 41.15 96.15)
@@
 	)
 	(segment
+		(start 41.1 94.5)
+		(end 40.5 94.5)
+		(width 0.2)
+		(layer "F.Cu")
+		(net "Net-(U35-IN+)")
+	)
+	(segment
 		(start 39.3 95.7)
 		(end 39.8 96.2)
@@
 	)
 	(segment
+		(start 55.11119 98.91119)
+		(end 53.5 97.3)
+		(width 0.2)
+		(layer "F.Cu")
+		(net "Net-(U35-IN+)")
+	)
+	(segment
+		(start 40.5 94.5)
+		(end 39.3 95.7)
+		(width 0.2)
+		(layer "F.Cu")
+		(net "Net-(U35-IN+)")
+	)
+	(segment
 		(start 39.8 96.2)
 		(end 41.1 96.2)
@@
 		(net "Net-(U35-IN+)")
 	)
+	(segment
+		(start 55.11119 109.71119)
+		(end 55.11119 98.91119)
+		(width 0.2)
+		(layer "F.Cu")
+		(net "Net-(U35-IN+)")
+	)
+	(via
+		(at 41.1 94.5)
+		(size 0.5)
+		(drill 0.25)
+		(layers "F.Cu" "B.Cu")
+		(net "Net-(U35-IN+)")
+	)
+	(via
+		(at 53.5 97.3)
+		(size 0.5)
+		(drill 0.25)
+		(layers "F.Cu" "B.Cu")
+		(net "Net-(U35-IN+)")
+	)
+	(segment
+		(start 41.7 93.9)
+		(end 41.1 94.5)
+		(width 0.2)
+		(layer "B.Cu")
+		(net "Net-(U35-IN+)")
+	)
+	(segment
+		(start 50.1 93.9)
+		(end 41.7 93.9)
+		(width 0.2)
+		(layer "B.Cu")
+		(net "Net-(U35-IN+)")
+	)
+	(segment
+		(start 53.5 97.3)
+		(end 50.1 93.9)
+		(width 0.2)
+		(layer "B.Cu")
+		(net "Net-(U35-IN+)")
+	)
