File: ScopeFun_PCB/file56948067.kicad_sch (KiCad schematic)
At the start: 26 parts, among them Q3 BSS138BKS, U12 XC7A35T-FTG256

Commit message: 0326
Parts:
- removed Q3: BSS138BKS, ScopefunPackagesLibrary:SOT363, symbol ScopefunParts:BSS138BKS
- removed R44, R57, R64: R_1.02k, ScopefunPackagesLibrary:R_0603, symbol ScopefunParts:R_1.02k
- added R41, R42, R65, R67: R_100, ScopefunPackagesLibrary:R_0402, symbol ScopefunParts:R_100
- SLP1, SLP2, SLP3: footprint ScopefunPackagesLibrary:SLP3-300-100-F -> ScopefunPackagesLibrary:SLP3-300-100-R
Connections:
- net CC_AB is gone; now on net RE7: U12.L12 (IO_L6P_T0_FCS_B_14)
- net ADCA_CS: now also U12.T7 (IO_L21P_T3_DQS_14); no longer U12.T8 (IO_L21N_T3_DQS_A06_D22_14)
- net ADC_SDIN: now also U12.T8 (IO_L21N_T3_DQS_A06_D22_14); no longer U12.T7 (IO_L21P_T3_DQS_14)
- net data1_N: now reaches U12.K13 (IO_L5P_T0_D06_14)
- net data1_N: now also R41.2
- net data1_P: now reaches U12.L13 (IO_L5N_T0_D07_14)
- net data1_P: now also R41.1
- net data12_N: now reaches U12.M6 (IO_L19P_T3_A10_D26_14)
- net data12_N: now also R65.2
- net data12_P: now reaches U12.N6 (IO_L19N_T3_A09_D25_VREF_14)
- net data12_P: now also R65.1
- net data11_P: now reaches U12.N9 (IO_L18P_T2_A12_D28_14)
- net data11_P: now also R42.2
- net data11_N: now reaches U12.P9 (IO_L18N_T2_A11_D27_14)
- net data11_N: now also R42.1
- net data13_P: now reaches U12.R5 (IO_L23P_T3_A03_D19_14)
- net data13_P: now also R67.2
- net data13_N: now reaches U12.T5 (IO_L23N_T3_A02_D18_14)
- net data13_N: now also R67.1
- net ADCB_CS: no longer names the net of U12.L15 (IO_L3P_T0_DQS_PUDC_B_14)
- net dataA0_N renamed data6_N
- net dataA0_P renamed data6_P
- net dataA1_N renamed data7_P
- net dataA1_P renamed data7_N
- net dataA2_N renamed data8_N
- net dataA2_P renamed data8_P
- net dataA3_N renamed data9_N
- net dataA3_P renamed data9_P
- net dataA4_N renamed data10_P
- net dataA4_P renamed data10_N
- net dataB0_N renamed data0_N
- net dataB0_P renamed data0_P
- net dataB1_N renamed data2_N
- net dataB1_P renamed data2_P
- net dataB2_N renamed data3_P
- net dataB2_P renamed data3_N
- net dataB3_N renamed data4_P
- net dataB3_P renamed data4_N
- net dataB4_N renamed data5_N
- net dataB4_P renamed data5_P
- no-connect marks 39 -> 32
Other:
- note removed: "PUDC_B = High I/Os 3-state during configuration"

Commit message: 260330
Connections:
- net data0_N: now also R54.2, U12.R10 (IO_L17P_T2_A14_D30_14); no longer R45.1, U12.K16 (IO_L2N_T0_D03_14)
- net data0_P: now also R54.1, U12.R11 (IO_L17N_T2_A13_D29_14); no longer R45.2, U12.K15 (IO_L2P_T0_D02_14)
- net data10_N: now also R67.2, U12.R5 (IO_L23P_T3_A03_D19_14); no longer R55.2, U12.T9 (IO_L22P_T3_A05_D21_14)
- net data10_P: now also R67.1, U12.T5 (IO_L23N_T3_A02_D18_14); no longer R55.1, U12.T10 (IO_L22N_T3_A04_D20_14)
- net data11_N: now also R55.2, U12.T9 (IO_L22P_T3_A05_D21_14); no longer R42.1, U12.P9 (IO_L18N_T2_A11_D27_14)
- net data11_P: now also R55.1, U12.T10 (IO_L22N_T3_A04_D20_14); no longer R42.2, U12.N9 (IO_L18P_T2_A12_D28_14)
- net data12_N: now also R42.1, U12.P9 (IO_L18N_T2_A11_D27_14); no longer R65.2, U12.M6 (IO_L19P_T3_A10_D26_14)
- net data12_P: now also R42.2, U12.N9 (IO_L18P_T2_A12_D28_14); no longer R65.1, U12.N6 (IO_L19N_T3_A09_D25_VREF_14)
- net data13_N: now also R65.2, U12.M6 (IO_L19P_T3_A10_D26_14); no longer R67.1, U12.T5 (IO_L23N_T3_A02_D18_14)
- net data13_P: now also R65.1, U12.N6 (IO_L19N_T3_A09_D25_VREF_14); no longer R67.2, U12.R5 (IO_L23P_T3_A03_D19_14)
- net data1_N: now also R49.1, U12.R16 (IO_L9N_T1_DQS_D13_14); no longer R41.2, U12.K13 (IO_L5P_T0_D06_14)
- net data1_P: now also R49.2, U12.R15 (IO_L9P_T1_DQS_14); no longer R41.1, U12.L13 (IO_L5N_T0_D07_14)
- net data4_N: now also R53.1, U12.T13 (IO_L16N_T2_A15_D31_14); no longer R48.2, U12.P15 (IO_L8P_T1_D11_14)
- net data4_P: now also R53.2, U12.R13 (IO_L16P_T2_CSI_B_14); no longer R48.1, U12.P16 (IO_L8N_T1_D12_14)
- net data5_N: now also R52.1, U12.P11 (IO_L14N_T2_SRCC_14); no longer R49.1, U12.R16 (IO_L9N_T1_DQS_D13_14)
- net data5_P: now also R52.2, U12.P10 (IO_L14P_T2_SRCC_14); no longer R49.2, U12.R15 (IO_L9P_T1_DQS_14)
- net data7_N: now also R41.2, U12.K13 (IO_L5P_T0_D06_14); no longer R53.2, U12.R13 (IO_L16P_T2_CSI_B_14)
- net data7_P: now also R41.1, U12.L13 (IO_L5N_T0_D07_14); no longer R53.1, U12.T13 (IO_L16N_T2_A15_D31_14)
- net data8_N: now also R45.1, U12.K16 (IO_L2N_T0_D03_14); no longer R52.1, U12.P11 (IO_L14N_T2_SRCC_14)
- net data8_P: now also R45.2, U12.K15 (IO_L2P_T0_D02_14); no longer R52.2, U12.P10 (IO_L14P_T2_SRCC_14)
- net data9_N: now also R48.2, U12.P15 (IO_L8P_T1_D11_14); no longer R54.1, U12.R11 (IO_L17N_T2_A13_D29_14)
- net data9_P: now also R48.1, U12.P16 (IO_L8N_T1_D12_14); no longer R54.2, U12.R10 (IO_L17P_T2_A14_D30_14)
Other:
- note added: "INVERTED POLARITY"
- note removed: "INVERTED POLARITY B1"

Commit message: 1
Connections:
- net data0_N: now also R52.2, U12.P10 (IO_L14P_T2_SRCC_14); no longer R54.2, U12.R10 (IO_L17P_T2_A14_D30_14)
- net data0_P: now also R52.1, U12.P11 (IO_L14N_T2_SRCC_14); no longer R54.1, U12.R11 (IO_L17N_T2_A13_D29_14)
- net data10_N: now also R42.1, U12.P9 (IO_L18N_T2_A11_D27_14); no longer R67.2, U12.R5 (IO_L23P_T3_A03_D19_14)
- net data10_P: now also R42.2, U12.N9 (IO_L18P_T2_A12_D28_14); no longer R67.1, U12.T5 (IO_L23N_T3_A02_D18_14)
- net data11_N: now also R65.2, U12.M6 (IO_L19P_T3_A10_D26_14); no longer R55.2, U12.T9 (IO_L22P_T3_A05_D21_14)
- net data11_P: now also R65.1, U12.N6 (IO_L19N_T3_A09_D25_VREF_14); no longer R55.1, U12.T10 (IO_L22N_T3_A04_D20_14)
- net data12_N: now also R67.1, U12.T5 (IO_L23N_T3_A02_D18_14); no longer R42.1, U12.P9 (IO_L18N_T2_A11_D27_14)
- net data12_P: now also R67.2, U12.R5 (IO_L23P_T3_A03_D19_14); no longer R42.2, U12.N9 (IO_L18P_T2_A12_D28_14)
- net data13_N: now also R55.1, U12.T10 (IO_L22N_T3_A04_D20_14); no longer R65.2, U12.M6 (IO_L19P_T3_A10_D26_14)
- net data13_P: now also R55.2, U12.T9 (IO_L22P_T3_A05_D21_14); no longer R65.1, U12.N6 (IO_L19N_T3_A09_D25_VREF_14)
- net data1_N: now also R53.2, U12.R13 (IO_L16P_T2_CSI_B_14); no longer R49.1, U12.R16 (IO_L9N_T1_DQS_D13_14)
- net data1_P: now also R53.1, U12.T13 (IO_L16N_T2_A15_D31_14); no longer R49.2, U12.R15 (IO_L9P_T1_DQS_14)
- net data4_N: now also R54.1, U12.R11 (IO_L17N_T2_A13_D29_14); no longer R53.1, U12.T13 (IO_L16N_T2_A15_D31_14)
- net data4_P: now also R54.2, U12.R10 (IO_L17P_T2_A14_D30_14); no longer R53.2, U12.R13 (IO_L16P_T2_CSI_B_14)
- net data5_N: now also R41.2, U12.K13 (IO_L5P_T0_D06_14); no longer R52.1, U12.P11 (IO_L14N_T2_SRCC_14)
- net data5_P: now also R41.1, U12.L13 (IO_L5N_T0_D07_14); no longer R52.2, U12.P10 (IO_L14P_T2_SRCC_14)
- net data6_N: now also R50.2, U12.T14 (IO_L10P_T1_D14_14); no longer R50.1, U12.T15 (IO_L10N_T1_D15_14)
- net data6_P: now also R50.1, U12.T15 (IO_L10N_T1_D15_14); no longer R50.2, U12.T14 (IO_L10P_T1_D14_14)
- net data7_N: now also R48.1, U12.P16 (IO_L8N_T1_D12_14); no longer R41.2, U12.K13 (IO_L5P_T0_D06_14)
- net data7_P: now also R48.2, U12.P15 (IO_L8P_T1_D11_14); no longer R41.1, U12.L13 (IO_L5N_T0_D07_14)
- net data8_N: now also R49.1, U12.R16 (IO_L9N_T1_DQS_D13_14); no longer R45.1, U12.K16 (IO_L2N_T0_D03_14)
- net data8_P: now also R49.2, U12.R15 (IO_L9P_T1_DQS_14); no longer R45.2, U12.K15 (IO_L2P_T0_D02_14)
- net data9_N: now also R45.2, U12.K15 (IO_L2P_T0_D02_14); no longer R48.2, U12.P15 (IO_L8P_T1_D11_14)
- net data9_P: now also R45.1, U12.K16 (IO_L2N_T0_D03_14); no longer R48.1, U12.P16 (IO_L8N_T1_D12_14)

Commit message: 260407
Connections:
- net data1_N: now also R53.1, U12.T13 (IO_L16N_T2_A15_D31_14); no longer R53.2, U12.R13 (IO_L16P_T2_CSI_B_14)
- net data1_P: now also R53.2, U12.R13 (IO_L16P_T2_CSI_B_14); no longer R53.1, U12.T13 (IO_L16N_T2_A15_D31_14)
- net data2_N: now also R45.1, U12.K16 (IO_L2N_T0_D03_14); no longer R47.2, U12.M16 (IO_L7P_T1_D09_14)
- net data2_P: now also R45.2, U12.K15 (IO_L2P_T0_D02_14); no longer R47.1, U12.N16 (IO_L7N_T1_D10_14)
- net data4_N: now also R41.2, U12.K13 (IO_L5P_T0_D06_14); no longer R54.1, U12.R11 (IO_L17N_T2_A13_D29_14)
- net data4_P: now also R41.1, U12.L13 (IO_L5N_T0_D07_14); no longer R54.2, U12.R10 (IO_L17P_T2_A14_D30_14)
- net data5_N: now also R49.1, U12.R16 (IO_L9N_T1_DQS_D13_14); no longer R41.2, U12.K13 (IO_L5P_T0_D06_14)
- net data5_P: now also R49.2, U12.R15 (IO_L9P_T1_DQS_14); no longer R41.1, U12.L13 (IO_L5N_T0_D07_14)
- net data8_N: now also R54.1, U12.R11 (IO_L17N_T2_A13_D29_14); no longer R49.1, U12.R16 (IO_L9N_T1_DQS_D13_14)
- net data8_P: now also R54.2, U12.R10 (IO_L17P_T2_A14_D30_14); no longer R49.2, U12.R15 (IO_L9P_T1_DQS_14)
- net data9_N: now also R47.2, U12.M16 (IO_L7P_T1_D09_14); no longer R45.2, U12.K15 (IO_L2P_T0_D02_14)
- net data9_P: now also R47.1, U12.N16 (IO_L7N_T1_D10_14); no longer R45.1, U12.K16 (IO_L2N_T0_D03_14)

Commit message: 260410
Connections:
- net dpot_cs: no longer names the net of U12.N11 (IO_L13P_T2_MRCC_14)
- net dpot_sck: no longer names the net of U12.P8 (IO_L20P_T3_A08_D24_14)
- net dpot_si: no longer names the net of U12.J13 (IO_L1P_T0_D00_MOSI_14)
- no-connect marks 32 -> 35
Changed lines of the file:
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@@
 	)
 	(no_connect
+		(at 73.66 124.46)
+	)
+	(no_connect
 		(at 149.86 147.32)
 	)
@@
 	)
 	(no_connect
+		(at 73.66 88.9)
+	)
+	(no_connect
 		(at 64.77 38.1)
 	)
@@
 	)
 	(no_connect
+		(at 73.66 27.94)
+	)
+	(no_connect
 		(at 189.23 33.02)
 	)
@@
 	(wire
 		(pts
-			(xy 72.39 124.46) (xy 73.66 124.46)
-		)
-		(stroke
-			(width 0)
-			(type default)
-		)
-	)
-	(wire
-		(pts
 			(xy 41.91 57.15) (xy 39.37 57.15)
 		)
@@
 	(wire
 		(pts
-			(xy 72.39 88.9) (xy 73.66 88.9)
-		)
-		(stroke
-			(width 0)
-			(type default)
-		)
-	)
-	(wire
-		(pts
 			(xy 53.34 138.43) (xy 53.34 137.16)
 		)
@@
 	(wire
 		(pts
-			(xy 68.58 27.94) (xy 73.66 27.94)
-		)
-		(stroke
-			(width 0)
-			(type default)
-		)
-	)
-	(wire
-		(pts
 			(xy 72.39 101.6) (xy 73.66 101.6)
 		)
@@
 		)
 	)
-	(global_label "dpot_cs"
-		(shape output)
-		(at 72.39 88.9 180)
-		(effects
-			(font
-				(size 1.27 1.27)
-			)
-			(justify right)
-		)
-		(property "Intersheetrefs" "${INTERSHEET_REFS}"
-			(at 72.39 88.9 0)
-			(effects
-				(font
-					(size 1.27 1.27)
-				)
-				(hide yes)
-			)
-		)
-	)
 	(global_label "data6_P"
 		(shape input)
@@
 		)
 	)
-	(global_label "dpot_si"
-		(shape output)
-		(at 68.58 27.94 180)
-		(effects
-			(font
-				(size 1.27 1.27)
-			)
-			(justify right)
-		)
-		(property "Intersheetrefs" "${INTERSHEET_REFS}"
-			(at 68.58 27.94 0)
-			(effects
-				(font
-					(size 1.27 1.27)
-				)
-				(hide yes)
-			)
-		)
-	)
 	(global_label "AN_TRIG_LEVEL"
 		(shape output)
@@
 			(effects
 				(font
-					(size 1.27 1.27)
-				)
-				(hide yes)
-			)
-		)
-	)
-	(global_label "dpot_sck"
-		(shape output)
-		(at 72.39 124.46 180)
-		(effects
-			(font
-				(size 1.27 1.27)
-			)
-			(justify right)
-		)
-		(property "Intersheetrefs" "${INTERSHEET_REFS}"
-			(at 72.39 124.46 0)
-			(effects
-				(font

Commit message: 260420
Other:
- moved on the sheet: LED1, LED2, LED3, R41, R42, R45, R46, R47, R48, R49, R50, R51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

Commit message: manufactured
Changed lines of the file:
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@@
 	(text "INVERTED\nPOLARITY CLK"
 		(exclude_from_sim no)
-		(at 31.75 86.36 0)
+		(at 32.258 87.122 0)
 		(effects
 			(font
