File: ScopeFun_PCB/file56948067.kicad_sch (KiCad schematic)
At the start: 26 parts, among them U12 XC7A35T-FTG256

Commit message: 0531
Parts:
- removed R56: R_100, ScopefunPackagesLibrary:R_0402, symbol ScopefunParts:R_100
Connections:
- net DASCLK: now reaches U12.M4 (IO_L1N_T0_34)
- net DASDIN: now reaches U12.N3 (IO_L3P_T0_DQS_34)
- net DASYNC: now reaches U12.N4 (IO_L6N_T0_VREF_34)
- net AN_TRIG_LEVEL: no longer names the net of U12.T12 (IO_L15N_T2_DQS_DOUT_CSO_B_14)
- net AN_TRIG_N: no longer names the net of U12.R7 (IO_L24N_T3_A00_D16_14)
- net AN_TRIG_P: no longer names the net of U12.R6 (IO_L24P_T3_A01_D17_14)
- net RE7: no longer names the net of U12.L12 (IO_L6P_T0_FCS_B_14)
- no-connect marks 35 -> 36
