File: ScopeFun_PCB/Scopefun_v3.kicad_sch (KiCad schematic)
At the start: 0 parts

Commit message: manufactured
Changed lines of the file:
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@@
 			)
 		)
-		(pin "CH1-" output
+		(pin "CH1-" input
 			(at 132.08 30.48 0)
 			(effects

Commit message: 0531
Other:
- added sheet CONTROL DAC (file58568C5C.kicad_sch)
Changed lines of the file:
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@@
+		)
+	)
+	(sheet
+		(at 209.55 25.4)
+		(size 46.99 16.51)
+		(exclude_from_sim no)
+		(in_bom yes)
+		(on_board yes)
+		(dnp no)
+		(fields_autoplaced yes)
+		(stroke
+			(width 0)
+			(type solid)
+		)
+		(fill
+			(color 0 0 0 0)
+		)
+		(property "Sheetname" "CONTROL DAC"
+			(at 209.55 24.0534 0)
+			(show_name no)
+			(do_not_autoplace no)
+			(effects
+				(font
+					(size 2.54 2.54)
+				)
+				(justify left bottom)
+			)
+		)
+		(property "Sheetfile" "file58568C5C.kicad_sch"
+			(at 209.55 42.4946 0)
+			(show_name no)
+			(do_not_autoplace no)
+			(effects
+				(font
+					(size 1.27 1.27)
+				)
+				(justify left top)
+			)
+		)
+		(instances
+			(project "Scopefun_v3"
+				(path "/29c98cb5-ff01-42d3-b159-4c21611d999f"
+					(page "3")
+				)
+			)
 		)
 	)
