File: ScopeFun_PCB/file56785EF9.kicad_sch (KiCad schematic)
At the start: 45 parts, among them U3 AD8337, U4 AD8337, U5 ADA4932-1, U6 ADA4932-1, U7 LTC6754

Commit message: 260412_2
Connections:
- net CH2_CM is gone; now on net CH_CM: C24.1, U6.9 (Vocm)
- net CH1_CM renamed CH_CM
Changed lines of the file:
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@@
 		)
 	)
-	(global_label "CH2_CM"
+	(global_label "CH_CM"
 		(shape input)
 		(at 147.32 151.13 180)
@@
 		)
 	)
-	(global_label "CH1_CM"
+	(global_label "CH_CM"
 		(shape input)
 		(at 147.32 63.5 180)

Commit message: 0531
Parts:
- removed C35, C36, C37: C_0.1u, ScopefunPackagesLibrary:C_0603, symbol ScopefunParts:C_0.1u
- removed D11: 1N4148W, ScopefunPackagesLibrary:SOD123, symbol ScopefunParts:1N4148W
- removed R31: R_499R, ScopefunPackagesLibrary:R_0603, symbol ScopefunParts:R_499R
- removed R36, R37: R_6.8k, ScopefunPackagesLibrary:R_0603, symbol ScopefunParts:R_6.8k
- removed RE7: G6K-2F-Y-DC4.5, ScopefunPackagesLibrary:G6K-2F-Y, symbol ScopefunParts:G6K-2F-Y-DC4.5
- removed U7: LTC6754, ScopefunPackagesLibrary:SC70-6, symbol ScopefunParts:LTC6754
Connections:
- net CH2_VGA: now also U4.3 (INPP)
- no-connect marks 3 -> 0
