File: ScopeFun_PCB/file58568C5C.kicad_sch (KiCad schematic)
At the start: 24 parts, among them U32A AZ4558C, U32B AZ4558C, U33 MAX5501, U34 OPA692, U35 OPA692

Commit message: 0531
Parts:
- removed U32A, U32B: AZ4558C, ScopefunPackagesLibrary:SOIC8, symbol ScopefunParts:AZ4558C
- added U7: AZ4558C, ScopefunPackagesLibrary:SOIC8, symbol ScopefunParts:AZ4558C
Connections:
- net -Va: now also U7.4 (V-), U7.4 (V-)
- net CH1_GAIN_ADJ: now also U7.5 (+)
- net CH2_GAIN_ADJ: now also U7.3 (+)
- net Va: now also U7.8 (V+), U7.8 (V+)
- net at R156.1, R158.2: now also U7.1
- net at R157.1, R159.2: now also U7.7
- net at R155.1, R157.2: now also U7.6 (-)
- net at R154.1, R156.2: now also U7.2 (-)
